Commit message: major updates of architechure

File: agro_cad/agrobot_description/urdf/agrobot.urdf (robot description, URDF)
Before this commit: robot agrobot, 20 links, 19 joints
Links:
- added link d435_link
- added link d435_link_optical
Joints:
- added joint d435_link_joint: type fixed, parent base_link, child d435_link, origin xyz=0.451636729 -0.017499974 0.691293991 rpy=0.000000000 0.872664626 0.000000000
- added joint d435_link_optical_joint: type fixed, parent d435_link, child d435_link_optical, origin xyz=0.000000000 0.000000000 0.000000000 rpy=-1.570796327 0.000000000 -1.570796327

File: agro_cad/agrobot_description/urdf/agrobot.urdf.xacro (robot description, xacro)
@@ -73,4 +73,18 @@
     <parent link="d405_link"/>
     <child link="d405_link_optical"/>
+    <origin xyz="0.000000000 0.000000000 0.000000000" rpy="-1.570796327 0.000000000 -1.570796327"/>
+  </joint>
+  <link name="d435_link">
+  </link>
+  <joint name="d435_link_joint" type="fixed">
+    <parent link="base_link"/>
+    <child link="d435_link"/>
+    <origin xyz="0.451636729 -0.017499974 0.691293991" rpy="0.000000000 0.872664626 0.000000000"/>
+  </joint>
+  <link name="d435_link_optical">
+  </link>
+  <joint name="d435_link_optical_joint" type="fixed">
+    <parent link="d435_link"/>
+    <child link="d435_link_optical"/>
     <origin xyz="0.000000000 0.000000000 0.000000000" rpy="-1.570796327 0.000000000 -1.570796327"/>
   </joint>

File: agro_cad/agrobot_frames.urdf (robot description, URDF)
Before this commit: robot agrobot, 10 links, 9 joints
Links:
- removed link zedm_center
- removed link zedm_center_optical
- removed link zedm_left
- removed link zedm_left_optical
- removed link zedm_right
- removed link zedm_right_optical
- added link d435_link
- added link d435_link_optical
- added link wheel_fl
- added link wheel_fr
- added link wheel_rl
- added link wheel_rr
Joints:
- removed joint zedm_center_joint
- removed joint zedm_center_optical_joint
- removed joint zedm_left_joint
- removed joint zedm_left_optical_joint
- removed joint zedm_right_joint
- removed joint zedm_right_optical_joint
- added joint d435_link_joint: type fixed, parent base_link, child d435_link, origin xyz=0.451636729 -0.017499974 0.691293991 rpy=0.000000000 0.872664626 0.000000000
- added joint d435_link_optical_joint: type fixed, parent d435_link, child d435_link_optical, origin xyz=0 0 0 rpy=-1.570796327 0.000000000 -1.570796327
- added joint wheel_fl_joint: type fixed, parent base_link, child wheel_fl, origin xyz=0.317800254 0.316000000 0.103505609 rpy=0.000000000 0.000000000 0.000000000
- added joint wheel_fr_joint: type fixed, parent base_link, child wheel_fr, origin xyz=0.317800254 -0.316000000 0.103505609 rpy=0.000000000 0.000000000 0.000000000
- added joint wheel_rl_joint: type fixed, parent base_link, child wheel_rl, origin xyz=-0.317800254 0.316000000 0.103505609 rpy=0.000000000 0.000000000 0.000000000
- added joint wheel_rr_joint: type fixed, parent base_link, child wheel_rr, origin xyz=-0.317800254 -0.316000000 0.103505609 rpy=0.000000000 0.000000000 0.000000000
